Commit message: updated yaml files

File: peg_lwr_robot/robot/peg_lwr_robot.urdf (robot description, URDF)
Before this commit: robot kuka_lwr_peg_robot, 18 links, 17 joints
Links:
- link dummy_link: geometry visual cylinder length=0.2 radius=0.01

Commit message: .

File: peg_lwr_robot/robot/peg_lwr_robot.urdf (robot description, URDF)
Before this commit: robot kuka_lwr_peg_robot, 18 links, 17 joints
Links:
- added link lwr_1_link_damping
- added link lwr_1_link_torque
- added link lwr_2_link_damping
- added link lwr_2_link_torque
- added link lwr_3_link_damping
- added link lwr_3_link_torque
- added link lwr_4_link_damping
- added link lwr_4_link_torque
- added link lwr_5_link_damping
- added link lwr_5_link_torque
- added link lwr_6_link_damping
- added link lwr_6_link_torque
- added link lwr_7_link_damping
- added link lwr_7_link_torque
Joints:
- removed joint target_frame
- removed joint target_frame_two
- added joint dummy_joint: type fixed, parent lwr_7_link, child dummy_link, origin xyz=0 0 0.2 rpy=0 0 0
- added joint lwr_0_joint_damping: type revolute, parent lwr_base_link, child lwr_1_link_damping, axis 0 0 1, limit lower=0 upper=500 effort=0 velocity=20000
- added joint lwr_0_joint_torque: type revolute, parent lwr_base_link, child lwr_1_link_torque, axis 0 0 1, limit lower=-2.96705972839 upper=2.96705972839 effort=176 velocity=1.91986217719
- added joint lwr_1_joint_damping: type revolute, parent lwr_1_link, child lwr_2_link_damping, axis 0 0 1, limit lower=0 upper=500 effort=0 velocity=20000
- added joint lwr_1_joint_torque: type revolute, parent lwr_1_link, child lwr_2_link_torque, axis 0 -1 0, limit lower=-2.09439510239 upper=2.09439510239 effort=176 velocity=1.91986217719
- added joint lwr_2_joint_damping: type revolute, parent lwr_2_link, child lwr_3_link_damping, axis 0 0 1, limit lower=0 upper=500 effort=0 velocity=20000
- added joint lwr_2_joint_torque: type revolute, parent lwr_2_link, child lwr_3_link_torque, axis 0 0 1, limit lower=0 upper=5000 effort=0 velocity=20000
- added joint lwr_3_joint_damping: type revolute, parent lwr_3_link, child lwr_4_link_damping, axis 0 0 1, limit lower=0 upper=500 effort=0 velocity=20000
- added joint lwr_3_joint_torque: type revolute, parent lwr_3_link, child lwr_4_link_torque, axis 0 1 0, limit lower=-2.09439510239 upper=2.09439510239 effort=100 velocity=2.23402144255
- added joint lwr_4_joint_damping: type revolute, parent lwr_4_link, child lwr_5_link_damping, axis 0 0 1, limit lower=0 upper=500 effort=0 velocity=20000
- added joint lwr_4_joint_torque: type revolute, parent lwr_4_link, child lwr_5_link_torque, axis 0 0 1, limit lower=0 upper=500 effort=0 velocity=20000
- added joint lwr_5_joint_damping: type revolute, parent lwr_5_link, child lwr_6_link_damping, axis 0 0 1, limit lower=0 upper=500 effort=0 velocity=20000
- added joint lwr_5_joint_torque: type revolute, parent lwr_5_link, child lwr_6_link_torque, axis 0 0 1, limit lower=0 upper=500 effort=0 velocity=20000
- added joint lwr_6_joint_damping: type revolute, parent lwr_6_link, child lwr_7_link_damping, axis 0 0 1, limit lower=0 upper=500 effort=0 velocity=20000
- added joint lwr_6_joint_torque: type revolute, parent lwr_6_link, child lwr_7_link_torque, axis 0 0 1, limit lower=0 upper=500 effort=0 velocity=20000
- added joint lwr_peg_joint: type fixed, parent dummy_link, child lwr_peg_link, origin xyz=0 0 0 rpy=0 0 0

File: peg_lwr_robot/robot/peg_lwr_robot.urdf.xacro (robot description, xacro)
@@ -7,6 +7,6 @@
 		<origin xyz="0 0 0" rpy="0 0 0"/>
 	</xacro:kuka_lwr>
-   	<joint name="target_frame" type="fixed">
-       		<origin xyz="0 0 0.2" rpy="0 1.57 0" />
+   	<joint name="dummy_joint" type="fixed">
+       		<origin xyz="0 0 0.2" rpy="0 0 0" />
        		<parent link="lwr_7_link" />
        		<child link="dummy_link" />
@@ -15,5 +15,5 @@
          	<origin xyz="0 0 0" rpy="0 0 0"/>
 		<visual>
-             		<origin xyz="0.12 0 0" rpy="0 ${M_PI / 2} 0"/>
+             		<origin xyz="0 0 -0.12" rpy="0 0 0"/>
              		<geometry>
 				<cylinder radius="0.01" length="0.2"/>
@@ -28,27 +28,27 @@
 		<material>Gazebo/Grey</material>
 	</gazebo>
-     	<joint name="target_frame_two" type="fixed">
-       		<origin xyz="0 0 0" rpy="0 0 3.14" />
+     	<joint name="lwr_peg_joint" type="fixed">
+       		<origin xyz="0 0 0" rpy="0 0 0" />
        		<parent link="dummy_link" />
        		<child link="lwr_peg_link" />
      	</joint>
 	<link name="lwr_peg_link">
-			<inertial>
-				<mass value="0.06"/>
-				<origin xyz="0 0 0"/>
-				<cuboid_inertia_def length="1" width="1" height="1" mass="0.06"/>
-			</inertial>
-        		<visual>
-             			<origin xyz="0 0 0" rpy="0 0 0"/>
-             			<geometry>
-                    			<mesh filename="package://peg_lwr_robot/meshes/peg.dae"/>
-             			</geometry>
-                	</visual>
-			<collision>
-	        	<origin xyz="0 0 0" rpy="0 0 0"/>
+    		<origin xyz="0 0 0" rpy="0 0 0"/>
+		<inertial>
+			<mass value="0.06"/>
+			<origin xyz="0 0 0"/>
+			<cuboid_inertia_def length="1" width="1" height="1" mass="0.06"/>
+		</inertial>
+        	<visual>
+             		<origin xyz="0 0 0" rpy="0 ${-M_PI/2} ${M_PI}"/>
+             		<geometry>
+               			<mesh filename="package://peg_lwr_robot/meshes/peg.dae"/>
+             		</geometry>
+               	</visual>
+         	<collision>
 			<geometry>
 				<cylinder radius="0.04" length="0.05"/>
 			</geometry>
-           		</collision>
+         	</collision>
 	</link>
 </robot>
